File: pcb-slim/pcb.kicad_pcb (KiCad board)
At the start: 2 copper layers, 285 x 92.5 mm, 90 parts, among them J1 OLED, U1 Elite-C

Commit message: Manual and bare case files
Routing:
- net VCC: track 142.1 -> 141.1 mm
Other:
- outline, holes or cut-outs redrawn
- board text added: "by dcpedit (rev 2) github.com/dcpedit/teeshirt"
- board text removed: "by dcpedit (rev 1) github.com/dcpedit/teeshirt"
