File: plate/plate.kicad_pcb (KiCad board)
At the start: 2 copper layers, 285 x 92.5 mm, 58 parts

Commit message: Case updates
Parts:
- removed the ? at (345.8, 121.1)
- removed the ? at (63.7, 121.1)
- removed H2 (x3): , 
- added HOLE: VAL**, hole:PKRHSL, F.Cu at (63.7, 121.1)
- added HOLE: VAL**, hole:PKRHSL, F.Cu at (345.8, 121.1)
Other:
- board size 285 x 92.5 mm -> 285 x 94.6 mm

Commit message: Add readme
Parts:
- removed the REF** at (238.1, 147.6)
- removed the REF** at (171.4, 147.6)
- REF**: moved to B.Cu
- turned REF** to 0 degrees
