File: plate-slim/plate-slim.kicad_pcb (KiCad board)
At the start: 2 copper layers, 285 x 92.5 mm, 58 parts

Commit message: Add readme
Parts:
- removed the REF** at (238.1, 147.6)
- removed the REF** at (171.4, 147.6)
- REF**: moved to B.Cu
- turned REF** to 0 degrees
